File: KiCad-PCB/aktivna_bass_gitara/aktivna_bass_gitara.kicad_pcb (KiCad board)
At the start: 2 copper layers, 80 x 55 mm, 84 parts, among them J1 Conn_01x02_Female, J2 Conn_01x02_Female, J3 Conn_01x02_Female, SW1 SW_SPDT, SW2 SW_SPDT, U1 TL074, U2 TL074

Commit message: v2
v2
Parts:
- added H1: MountingHole, MountingHole:MountingHole_3.2mm_M3, F.Cu at (115.5, 84.5)
- added H2: MountingHole, MountingHole:MountingHole_3.2mm_M3, F.Cu at (44.5, 84.5)
- added H3: MountingHole, MountingHole:MountingHole_3.2mm_M3, F.Cu at (115.5, 130.5)
- added H4: MountingHole, MountingHole:MountingHole_3.2mm_M3, F.Cu at (44.5, 130.5)
- R25: footprint Resistor_THT:R_Axial_DIN0207_L6.3mm_D2.5mm_P7.62mm_Horizontal -> Resistor_THT:R_Axial_DIN0204_L3.6mm_D1.6mm_P5.08mm_Horizontal
- R6: moved to B.Cu
- moved R25 3.14 mm to (70.1, 91.1), turned to 90 degrees
- moved R40 2.30 mm to (105.8, 124.7)
- moved SW1 2.25 mm to (52.3, 89.3)
- moved R41 1.85 mm to (113.6, 124.7), turned to 180 degrees
- moved C16 1.30 mm to (83.3, 104.6)
- moved JP1 0.76 mm to (86.1, 99.6)
Routing:
- net Net-(R25-Pad2): track 50.7 -> 73.6 mm
- net VDC: track 134.6 -> 120.8 mm
- net Net-(C10-Pad2): track 3.86 -> 10.9 mm
- net Net-(C16-Pad1): track 18.8 -> 12.3 mm
- net Net-(C23-Pad1): track 41.2 -> 35.4 mm
- net Net-(C20-Pad2): track 28.4 -> 33.3 mm
- net Net-(R33-Pad1): track 4.08 -> 8.27 mm
- net Net-(C12-Pad2): track 8.42 -> 12.4 mm
- net GND: track 289.3 -> 293.0 mm
- net Net-(RV1-Pad2): track 40.9 -> 37.7 mm
- net Net-(C21-Pad2): track 23.6 -> 21.3 mm
- net Net-(R32-Pad1): track 41.4 -> 43.7 mm
- net Net-(R25-Pad1): track 22.0 -> 19.8 mm
- net Net-(C21-Pad1): track 34.6 -> 32.8 mm
- net Net-(C16-Pad2): track 11.7 -> 13.5 mm
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- added copper zone on F.Cu, net Net-(C12-Pad2)
- added copper zone on F.Cu, net Net-(C22-Pad2)
- added copper zone on F.Cu, net Net-(C8-Pad2)
- added copper zone on F.Cu, net VDC

Commit message: v3
v3
Parts:
- C19: footprint Capacitor_SMD:C_0805_2012Metric_Pad1.18x1.45mm_HandSolder -> Capacitor_THT:C_Rect_L7.0mm_W2.0mm_P5.00mm; moved to B.Cu
- C20, C4: footprint Capacitor_SMD:C_0805_2012Metric_Pad1.18x1.45mm_HandSolder -> Capacitor_THT:C_Disc_D3.0mm_W1.6mm_P2.50mm; moved to B.Cu
- moved R42 1.94 mm to (112.4, 116.0)
- moved RV5 1.84 mm to (114.6, 121.4)
- moved C19 1.82 mm to (104.2, 110.4)
- moved C20 1.57 mm to (89.2, 102.3)
- moved C4 1.53 mm to (59.4, 100.6)
- moved RT2 1.14 mm to (101.5, 119.1)
- moved R35 0.89 mm to (101.7, 110.9)
Routing:
- net Net-(R33-Pad1): track 8.27 -> 3.04 mm
- net Net-(C19-Pad2): track 14.2 -> 11.2 mm
- net Net-(C21-Pad2): track 21.3 -> 19.9 mm
- net Net-(R41-Pad2): track 3.39 -> 4.16 mm
- net Net-(C21-Pad1): track 32.8 -> 32.0 mm
- net Net-(R42-Pad1): track 6.32 -> 6.96 mm

Commit message: V4
Other:
- board text added: "By Ivan Hotovec 10/05/2021"
