File: KiCad-PCB/aktivna_bass_gitara/aktivna_bass_gitara.sch (KiCad schematic (older format))
At the start: 84 parts, among them J1 Conn_01x02_Female, J2 Conn_01x02_Female, J3 Conn_01x02_Female, SW1 SW_SPDT, SW2 SW_SPDT, U1 TL074, U2 TL074

Commit message: v2
v2
Parts:
- added H1, H2, H3, H4: MountingHole, MountingHole:MountingHole_3.2mm_M3, symbol Mechanical:MountingHole
- R25: footprint Resistor_THT:R_Axial_DIN0207_L6.3mm_D2.5mm_P7.62mm_Horizontal -> Resistor_THT:R_Axial_DIN0204_L3.6mm_D1.6mm_P5.08mm_Horizontal
Changed lines of the file:
@@
 F 0 "R25" V 14657 4300 50  0000 C CNN
 F 1 "3.3k" V 14566 4300 50  0000 C CNN
-F 2 "Resistor_THT:R_Axial_DIN0207_L6.3mm_D2.5mm_P7.62mm_Horizontal" V 14380 4300 50  0001 C CNN
+F 2 "Resistor_THT:R_Axial_DIN0204_L3.6mm_D1.6mm_P5.08mm_Horizontal" V 14380 4300 50  0001 C CNN
 F 3 "~" H 14450 4300 50  0001 C CNN
 	1    14450 4300
@@
 	-1   0    0    1
 $EndComp
+$Comp
+L Mechanical:MountingHole H1
+U 1 1 6162AC38
+P 6500 10250
+F 0 "H1" H 6600 10296 50  0000 L CNN
+F 1 "MountingHole" H 6600 10205 50  0000 L CNN
+F 2 "MountingHole:MountingHole_3.2mm_M3" H 6500 10250 50  0001 C CNN
+F 3 "~" H 6500 10250 50  0001 C CNN
+	1    6500 10250
+	1    0    0    -1
+$EndComp
+$Comp
+L Mechanical:MountingHole H2
+U 1 1 6162B5EF
+P 6500 10550
+F 0 "H2" H 6600 10596 50  0000 L CNN
+F 1 "MountingHole" H 6600 10505 50  0000 L CNN
+F 2 "MountingHole:MountingHole_3.2mm_M3" H 6500 10550 50  0001 C CNN
+F 3 "~" H 6500 10550 50  0001 C CNN
+	1    6500 10550
+	1    0    0    -1
+$EndComp
+$Comp
+L Mechanical:MountingHole H3
+U 1 1 61637A88
+P 7450 10200
+F 0 "H3" H 7550 10246 50  0000 L CNN
+F 1 "MountingHole" H 7550 10155 50  0000 L CNN
+F 2 "MountingHole:MountingHole_3.2mm_M3" H 7450 10200 50  0001 C CNN
+F 3 "~" H 7450 10200 50  0001 C CNN
+	1    7450 10200
+	1    0    0    -1
+$EndComp
+$Comp
+L Mechanical:MountingHole H4
+U 1 1 61643EEB
+P 7500 10600
+F 0 "H4" H 7600 10646 50  0000 L CNN
+F 1 "MountingHole" H 7600 10555 50  0000 L CNN
+F 2 "MountingHole:MountingHole_3.2mm_M3" H 7500 10600 50  0001 C CNN
+F 3 "~" H 7500 10600 50  0001 C CNN
+	1    7500 10600
+	1    0    0    -1
+$EndComp
 $EndSCHEMATC

Commit message: v3
v3
Parts:
- C19: footprint Capacitor_SMD:C_0805_2012Metric_Pad1.18x1.45mm_HandSolder -> Capacitor_THT:C_Rect_L7.0mm_W2.0mm_P5.00mm
- C20, C4: footprint Capacitor_SMD:C_0805_2012Metric_Pad1.18x1.45mm_HandSolder -> Capacitor_THT:C_Disc_D3.0mm_W1.6mm_P2.50mm
Changed lines of the file:
@@
 F 0 "C4" H 3535 4304 50  0000 R CNN
 F 1 "220p" H 3535 4395 50  0000 R CNN
-F 2 "Capacitor_SMD:C_0805_2012Metric_Pad1.18x1.45mm_HandSolder" H 3688 4200 50  0001 C CNN
+F 2 "Capacitor_THT:C_Disc_D3.0mm_W1.6mm_P2.50mm" H 3688 4200 50  0001 C CNN
 F 3 "~" H 3650 4350 50  0001 C CNN
 	1    3650 4350
@@
 F 0 "C20" V 16748 5050 50  0000 C CNN
 F 1 "220p" V 16839 5050 50  0000 C CNN
-F 2 "Capacitor_SMD:C_0805_2012Metric_Pad1.18x1.45mm_HandSolder" H 17038 4900 50  0001 C CNN
+F 2 "Capacitor_THT:C_Disc_D3.0mm_W1.6mm_P2.50mm" H 17038 4900 50  0001 C CNN
 F 3 "~" H 17000 5050 50  0001 C CNN
 	1    17000 5050
@@
 F 0 "C19" H 16015 6846 50  0000 L CNN
 F 1 "1n" H 16015 6755 50  0000 L CNN
-F 2 "Capacitor_SMD:C_0805_2012Metric_Pad1.18x1.45mm_HandSolder" H 15938 6650 50  0001 C CNN
+F 2 "Capacitor_THT:C_Rect_L7.0mm_W2.0mm_P5.00mm" H 15938 6650 50  0001 C CNN
 F 3 "~" H 15900 6800 50  0001 C CNN
 	1    15900 6800

Commit message: V4
Parts:
- C10, C11, C13, C6, C7, C9: value 68n -> 100n
- C21, C23: value 4.7u -> 2.2n; symbol Device:CP_Small -> Device:C
- R15, R21: value 220k -> 270k
- R43: value 2.7k -> 2.8k
Other:
- note added: "Bass & Treble"
- note added: "Buffer"
- note added: "Connectors"
- note added: "Equilizer"
- note added: "HighPass Filter"
- note added: "Input/Gain stage"
- note added: "Middle"
- note added: "Mounting Holes"
- note added: "OpAmp Power"
- note added: "PREDPOJAČALO ZA AKTIVNU BASS GITARU"
- moved on the sheet: C1, C10, C11, C12, C13, C14, C15, C16, C17, C18, C19, C2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
